Commit message: update description with camera_link

File: magni_description/urdf/magni.urdf.xacro (robot description, xacro)
@@ -147,3 +147,9 @@
     </xacro:raspi_camera>
   </xacro:if>
+  <link name="camera_link"/>
+  <joint name="camera_link_joint" type="fixed">
+    <parent link="base_link"/>
+    <child link="camera_link"/>
+    <origin xyz="0.00 0.00 0.16" rpy="0.0174533 -0.226893 0" />
+  </joint>
 </robot>
